File: v1/HWDesign/EAGLE/bluz_gw_shield_v1_revD.sch (EAGLE design)
At the start: 20 parts, among them J2 USB-MICROB, Q1 FC-12M, U2 MDBT40SMD, U3 SST25VF040B-S2, U4 SPARK_CORE

Commit message: newest files from adding the LED on D7 and TX/RX pins
Parts:
- removed U3: SST25VF040B-S2, Spark:SST25VF040B-S2
- added L2: (no value), led:LEDCHIP-LED0603
- added R3: 1k, SparkFun-Passives:RESISTOR0603-RES
- added U5: SST25VF010A-33-4I-SAE, Silicon_Storage_Tech_By_element14_Batch_1:SST25VF010A-33-4I-SAE
- renumbered LED1 to L1
Connections:
- removed net D0: JP6.8, U2.P0.00
- removed net D1: JP6.7, U2.P0.01
- new net N$10: U4.D1
- new net N$11: U4.D2
- new net N$12: U4.D3
- new net N$13: U4.D4
- new net N$14: U4.D5
- new net N$15: U4.D6
- new net N$16: U4.D7
- new net N$17: U4.VDDA
- new net N$2: L2.A, R3.2
- new net N$3: U4.A7
- new net N$4: U4.A1
- new net N$6: U4.A0
- new net N$9: U4.D0
- new net NRF_RX: JP6.2, U2.P0.06
- new net NRF_TX: JP6.1, U2.P0.07
- net D2: now also JP6.3, U2.P0.05; no longer JP6.6, U2.P0.02
- net D3: now also JP6.4, U2.P0.04; no longer JP6.5, U2.P0.03
- net D4: now also JP6.5, U2.P0.03; no longer JP6.4, U2.P0.04
- net D5: now also JP6.6, U2.P0.02; no longer JP6.3, U2.P0.05
- net D6: now also JP6.7, U2.P0.01; no longer JP6.2, U2.P0.06
- net D7: now also JP6.8, R3.1, U2.P0.00; no longer JP6.1, U2.P0.07
- net GND: now also L2.C, U5.VSS; no longer U3.VSS
- net SPI_MISO: now also U5.SO; no longer U3.SO
- net SPI_MOSI: now also U5.SI; no longer U3.SI
- net SPI_SCK: now also U5.SCK; no longer U3.SCK
- net SPI_SS: now also U5.CE; no longer U3.CE
- net VCC: now also U5.HOLD, U5.VDD, U5.WP; no longer U3.HOLD, U3.VDD, U3.WP
Other:
- note added: "D"
- note removed: "C"
- note removed: "J1"
